Commit message: feat: improve path and LiDAR visualization

File: src/ioniq5_description/urdf/ioniq5_base.xacro (robot description, xacro)
@@ -4,28 +4,72 @@
     <xacro:property name="length" value="${specs['dimensions']['length_m']}"/>
     <xacro:property name="width" value="${specs['dimensions']['width_m']}"/>
-    <xacro:property name="height" value="${specs['dimensions']['height_m']}"/>
+    <xacro:property name="wheelbase" value="${specs['dimensions']['wheelbase_m']}"/>
+    <xacro:property name="front_overhang" value="${specs['dimensions']['front_overhang_m']}"/>
+    <xacro:property name="rear_overhang" value="${specs['dimensions']['rear_overhang_m']}"/>
+    <xacro:property name="body_height" value="${specs['visualization']['body_height_m']}"/>
+    <xacro:property name="rear_axle_height" value="${specs['visualization']['rear_axle_height_m']}"/>
+    <xacro:property name="wheel_radius" value="${specs['visualization']['wheel_radius_m']}"/>
+    <xacro:property name="wheel_width" value="${specs['visualization']['wheel_width_m']}"/>
+    <xacro:property name="body_center_x" value="${(wheelbase + front_overhang - rear_overhang) / 2.0}"/>
+    <xacro:property name="body_center_z" value="${body_height / 2.0 - rear_axle_height}"/>
+    <xacro:property name="wheel_center_y" value="${width / 2.0 - wheel_width / 2.0}"/>
     <material name="ioniq5_body_color">
       <color rgba="0.55 0.62 0.67 0.75"/>
     </material>
+    <material name="ioniq5_wheel_color">
+      <color rgba="0.05 0.05 0.05 1.0"/>
+    </material>
     <link name="base_footprint"/>
     <link name="base_link">
-      <visual>
-        <origin xyz="0 0 ${height / 2.0}" rpy="0 0 0"/>
+      <!--
+        MORAI vehicle-local origin is the rear-axle center. The debug body
+        therefore extends from -rear_overhang to wheelbase+front_overhang.
+      -->
+      <visual name="body">
+        <origin xyz="${body_center_x} 0 ${body_center_z}" rpy="0 0 0"/>
         <geometry>
-          <box size="${length} ${width} ${height}"/>
+          <box size="${length} ${width} ${body_height}"/>
         </geometry>
         <material name="ioniq5_body_color"/>
       </visual>
-      <collision>
-        <origin xyz="0 0 ${height / 2.0}" rpy="0 0 0"/>
+      <collision name="body_collision">
+        <origin xyz="${body_center_x} 0 ${body_center_z}" rpy="0 0 0"/>
         <geometry>
-          <box size="${length} ${width} ${height}"/>
+          <box size="${length} ${width} ${body_height}"/>
         </geometry>
       </collision>
+      <visual name="rear_left_wheel">
+        <origin xyz="0 ${wheel_center_y} 0" rpy="${pi / 2.0} 0 0"/>
+        <geometry>
+          <cylinder radius="${wheel_radius}" length="${wheel_width}"/>
+        </geometry>
+        <material name="ioniq5_wheel_color"/>
+      </visual>
+      <visual name="rear_right_wheel">
+        <origin xyz="0 ${-wheel_center_y} 0" rpy="${pi / 2.0} 0 0"/>
+        <geometry>
+          <cylinder radius="${wheel_radius}" length="${wheel_width}"/>
+        </geometry>
+        <material name="ioniq5_wheel_color"/>
+      </visual>
+      <visual name="front_left_wheel">
+        <origin xyz="${wheelbase} ${wheel_center_y} 0" rpy="${pi / 2.0} 0 0"/>
+        <geometry>
+          <cylinder radius="${wheel_radius}" length="${wheel_width}"/>
+        </geometry>
+        <material name="ioniq5_wheel_color"/>
+      </visual>
+      <visual name="front_right_wheel">
+        <origin xyz="${wheelbase} ${-wheel_center_y} 0" rpy="${pi / 2.0} 0 0"/>
+        <geometry>
+          <cylinder radius="${wheel_radius}" length="${wheel_width}"/>
+        </geometry>
+        <material name="ioniq5_wheel_color"/>
+      </visual>
     </link>
     <joint name="base_footprint_to_base_link" type="fixed">
       <parent link="base_footprint"/>
       <child link="base_link"/>
-      <origin xyz="0 0 0" rpy="0 0 0"/>
+      <origin xyz="0 0 ${rear_axle_height}" rpy="0 0 0"/>
     </joint>
   </xacro:macro>

File: src/ioniq5_description/urdf/molit_sensors.xacro (robot description, xacro)
@@ -55,4 +55,28 @@
     </joint>
   </xacro:macro>
+  <xacro:macro name="lidar_sensor_mount" params="config parent">
+    <xacro:property name="xyz" value="${config['xyz_m']}"/>
+    <xacro:property name="rpy" value="${config['rpy_deg']}"/>
+    <link name="${config['frame_id']}">
+      <!-- VLP 계열 센서의 위치와 방향을 확인하기 위한 RViz용 단순 형상 -->
+      <visual name="lidar_body">
+        <origin xyz="0 0 0.035" rpy="0 0 0"/>
+        <geometry><cylinder radius="0.052" length="0.070"/></geometry>
+        <material name="lidar_body_color"><color rgba="0.08 0.22 0.35 1.0"/></material>
+      </visual>
+      <visual name="lidar_window">
+        <origin xyz="0 0 0.075" rpy="0 0 0"/>
+        <geometry><cylinder radius="0.050" length="0.025"/></geometry>
+        <material name="lidar_window_color"><color rgba="0.10 0.75 0.95 0.95"/></material>
+      </visual>
+    </link>
+    <joint name="${parent}_to_${config['frame_id']}" type="fixed">
+      <parent link="${parent}"/>
+      <child link="${config['frame_id']}"/>
+      <origin
+        xyz="${xyz[0]} ${xyz[1]} ${xyz[2]}"
+        rpy="${rpy[0] * pi / 180.0} ${rpy[1] * pi / 180.0} ${rpy[2] * pi / 180.0}"/>
+    </joint>
+  </xacro:macro>
   <xacro:macro name="molit_sensor_mounts" params="mounts">
     <xacro:property name="parent" value="${mounts['reference_frame']}"/>
@@ -67,5 +91,5 @@
     </xacro:if>
     <xacro:if value="${mounts['lidar']['transform_verified']}">
-      <xacro:generic_sensor_mount config="${mounts['lidar']}" parent="${parent}"/>
+      <xacro:lidar_sensor_mount config="${mounts['lidar']}" parent="${parent}"/>
     </xacro:if>
   </xacro:macro>
